File: Design_IoT_v3/IoTSchem.brd (EAGLE design)
At the start: 76.2 x 76.2 mm, 58 parts, among them IC1 DHT22, IC2 LM2596S, J1 SIM7000A, J2 BM06B-SRSS-TB, J4 640456-2, J5 640456-2, J6 640456-2, U1 ESP32-WROVER-E-N4R8, U2 MCP73831, U5 CH340C

Commit message: as sent to board house
Parts:
- moved R6 8.38 mm to (29.7, 38.9), turned to 0 degrees
- moved C1 4.83 mm to (34.0, 36.6), turned to 180 degrees
- moved C18 4.33 mm to (29.7, 36.6), turned to 180 degrees
- moved R4 2.70 mm to (38.6, 38.9)
- moved R5 2.27 mm to (34.0, 38.9), turned to 0 degrees
- moved R7 0.25 mm to (11.2, 14.0)
- moved C11 0.25 mm to (32.0, 10.2)
- moved R17 0.25 mm to (23.9, 10.2)
Connections:
- net BATT_SENSE: now also U1.6; no longer U1.12
- net BOOT: now also U5.13
- net RESET: now also U5.14
- net TEMP_SENSE: now also U1.7; no longer U1.13
Routing:
- net RESET: track 51.8 -> 100.5 mm, vias 2 -> 4
- net BOOT: track 19.7 -> 61.2 mm, vias 2 -> 4
- net TEMP_SENSE: track 34.4 -> 48.9 mm
- net BATT_SENSE: track 13.7 -> 7.67 mm
- net +3V7: track 103.7 -> 102.7 mm
- net D-: track 18.3 -> 17.7 mm
- net TX: track 62.2 -> 62.7 mm
Other:
- board text added: "Software Logistics, LLC NuvIoT Remote Sensing Board RSB-003 REV001 - 2022-10-03"
