File: Design_IoT_v3/IoTSchem.sch (EAGLE design)
At the start: 58 parts, among them IC1 DHT22, IC2 LM2596S, IC3 LM1117MPX-3.3, J1 SIM7000A, J2 BM06B-SRSS-TB, J4 640456-2, J5 640456-2, J6 640456-2, U1 ESP32-WROVER-E-N4R8, U2 MCP73831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

Commit message: Add files via upload
Parts:
- C1, C18: DIGIKEYPART# (none) -> 311-1365-1-ND
- C10: DIGIKEYPART# (none) -> 399-C0805C106K8PAC7800CT-ND
- C11, C7: DIGIKEYPART# (none) -> 311-1140-1-ND
- C12: DIGIKEYPART# (none) -> 1276-1015-1-ND
- C2, C3, C5: DIGIKEYPART# (none) -> 1276-6722-1-ND
- IC1: DIGIKEYPART# (none) -> 1528-1504-ND
- IC2: DIGIKEYPART# (none) -> 2156-LM2596SX-5.0/NOPB-ND
- IC3: DIGIKEYPART# (none) -> LM1117IMP-3.3/NOPBCT-ND
- IC4: DIGIKEYPART# (none) -> 893-1181-1-ND
- R10, R13, R14, R4, R5: DIGIKEYPART# (none) -> RMCF0805FT2K00CT-ND
- R11, R12, R2, R3, R6, R7, R8: DIGIKEYPART# (none) -> RMCF0805JT330RCT-ND
- R16, R17: DIGIKEYPART# (none) -> RMCF0805JT5K10CT-ND
- U2: DIGIKEYPART# (none) -> MCP73831T-2DCI/OTCT-ND

Commit message: as sent to board house
Connections:
- net BATT_SENSE: now also U1.IO34; no longer U1.IO27
- net BOOT: now also U5.!DTR
- net RESET: now also U5.!RTS
- net TEMP_SENSE: now also U1.IO35; no longer U1.IO14
Changed lines of the file:
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@@
 <wire x1="106.68" y1="109.22" x2="114.3" y2="109.22" width="0.1524" layer="91"/>
+</segment>
+<segment>
+<pinref part="U5" gate="U1" pin="!RTS"/>
+<wire x1="111.76" y1="38.1" x2="124.46" y2="38.1" width="0.1524" layer="91"/>
+<label x="114.3" y="38.1" size="1.778" layer="95"/>
 </segment>
 </net>
@@
 <wire x1="175.26" y1="58.42" x2="182.88" y2="58.42" width="0.1524" layer="91"/>
 <label x="177.8" y="58.42" size="1.778" layer="95"/>
+</segment>
+<segment>
+<pinref part="U5" gate="U1" pin="!DTR"/>
+<wire x1="111.76" y1="35.56" x2="124.46" y2="35.56" width="0.1524" layer="91"/>
+<label x="114.3" y="35.56" size="1.778" layer="95"/>
 </segment>
 </net>
@@
 </segment>
 <segment>
-<pinref part="U1" gate="A" pin="IO14"/>
-<wire x1="129.54" y1="83.82" x2="116.84" y2="83.82" width="0.1524" layer="91"/>
-<label x="109.22" y="83.82" size="1.778" layer="95"/>
+<pinref part="U1" gate="A" pin="IO35"/>
+<wire x1="129.54" y1="99.06" x2="116.84" y2="99.06" width="0.1524" layer="91"/>
+<label x="111.76" y="99.06" size="1.778" layer="95"/>
 </segment>
 </net>
@@
 </segment>
 <segment>
-<label x="114.3" y="40.64" size="1.27" layer="95" font="vector" xref="yes"/>
-<wire x1="111.76" y1="40.64" x2="113.03" y2="40.64" width="0.1524" layer="91"/>
+<label x="124.46" y="40.64" size="1.27" layer="95" font="vector" xref="yes"/>
+<wire x1="111.76" y1="40.64" x2="123.19" y2="40.64" width="0.1524" layer="91"/>
 <pinref part="U5" gate="U1" pin="RXI"/>
 <pinref part="D4" gate="G$1" pin="C"/>
-<wire x1="113.03" y1="40.64" x2="114.3" y2="40.64" width="0.1524" layer="91"/>
+<wire x1="123.19" y1="40.64" x2="124.46" y2="40.64" width="0.1524" layer="91"/>
 <wire x1="128.27" y1="39.37" x2="123.19" y2="39.37" width="0.1524" layer="91"/>
-<wire x1="123.19" y1="39.37" x2="123.19" y2="36.83" width="0.1524" layer="91"/>
-<wire x1="123.19" y1="36.83" x2="113.03" y2="36.83" width="0.1524" layer="91"/>
-<wire x1="113.03" y1="36.83" x2="113.03" y2="40.64" width="0.1524" layer="91"/>
-<junction x="113.03" y="40.64"/>
+<wire x1="123.19" y1="39.37" x2="123.19" y2="40.64" width="0.1524" layer="91"/>
+<junction x="123.19" y="40.64"/>
 </segment>
 </net>
@@
 </segment>
 <segment>
-<pinref part="U1" gate="A" pin="IO27"/>
-<wire x1="129.54" y1="86.36" x2="116.84" y2="86.36" width="0.1524" layer="91"/>
-<label x="109.22" y="86.36" size="1.778" layer="95"/>
-</segment>
-</net>
+<pinref part="U1" gate="A" pin="IO34"/>
+<wire x1="129.54" y1="101.6" x2="116.84" y2="101.6" width="0.1524" layer="91"/>
+<label x="111.76" y="101.6" size="1.778" layer="95"/>
+</segment>
+</net>
